File: kicad/transistor_tester.sch (KiCad schematic (older format))
At the start: 15 parts, among them IC1 ATTINY88-A, P1 PROG, P2 TEST, Q1 BSS138, Q2 BSS138, Q3 BSS138, SW1 SW_PUSH

Commit message: [README]: description + images + tidy up schematics.
Parts:
- BT1: symbol Battery -> Battery-RESCUE-transistor_tester
- Q1, Q2, Q3: symbol BSS138 -> BSS138-RESCUE-transistor_tester
